File: GatewayPlus_V1.1.kicad_pcb (KiCad board)
At the start: 2 copper layers, 100 x 67 mm, 207 parts, among them IC1 MP1584EN, IC2 MP1584EN, J1 LTDC_LCD_FPC_40p, J10 USB_OTG, J11 USB_WIFI_FLASH, J2 Micro_SD_Card, J3 ESP Anten, J4 xAnt2, J5 HR911105A, J6 RS485, J7 Conn_Jack-DC, J8 AudioJack4, J9 xAnt1, SW1 SW_Push, SW2 ESP_RESET, SW3 ESP_BOOT, U1 STM32F429IGTx, U2 IS42S16400J - HY57V641620E, U3 W25Q128JVS, U4 ESP32-D0WD-V3, U5 W25Q32JVSS, U6 Ai-Thinker-Ra-02, U7 LAN8720A, U8 MAX485E, X1 50MHz, Y1 32.768KHz, Y2 25MHz, Y3 40MHz

Commit message: Finish SDRAM, LCD, Power block.
Parts:
- added C89: 10uF, Capacitor_SMD:C_1206_3216Metric, F.Cu at (174.7, 126.9)
- added U9: CP2102N-Axx-xQFN28, Package_DFN_QFN:QFN-28-1EP_5x5mm_P0.5mm_EP3.35x3.35mm, F.Cu at (187.6, 111.7)
- J2: moved to F.Cu
- moved U6 119.1 mm to (79.2, 132.9)
- moved R47 64.6 mm to (166.2, 66.8), turned to -90 degrees
- moved JP7 60.9 mm to (141.3, 126.7), turned to 0 degrees
- moved R48 60.6 mm to (164.9, 66.8), turned to 90 degrees
- moved JP6 59.3 mm to (141.3, 125.4), turned to 0 degrees
- moved C69 59.1 mm to (119.4, 124.8)
- moved C32 59.1 mm to (126.9, 115.8)
- moved C33 59.1 mm to (137.5, 115.8)
- moved C62 59.1 mm to (132.4, 115.8)
- moved C65 59.1 mm to (122.1, 115.0)
- moved C66 59.1 mm to (122.1, 116.5)
- moved C68 59.1 mm to (136.2, 115.8)
- moved L3 59.1 mm to (124.4, 115.8)
- moved R13 59.1 mm to (133.7, 115.8)
- moved R19 59.1 mm to (134.9, 115.8)
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Connections:
- D7 pad 1: GND -> Net-(D6-Pad1)
- D7 pad 2: Net-(D6-Pad1) -> GND
Routing:
- net +3.3V: track 177.2 -> 361.9 mm, vias 17 -> 25
- net GND: track 43.3 -> 117.6 mm, vias 9 -> 19
- net /LTDC TFT LCD/LTDC_R5: track 0.00 -> 53.9 mm, vias 0 -> 2
- net /LTDC TFT LCD/LTDC_R1: track 0.00 -> 53.9 mm, vias 0 -> 2
- net /LTDC TFT LCD/LTDC_R0: track 0.00 -> 51.9 mm, vias 0 -> 2
- net /LTDC TFT LCD/LTDC_R6: track 0.00 -> 50.9 mm, vias 0 -> 2
- net /LTDC TFT LCD/LTDC_R3: track 0.00 -> 49.8 mm, vias 0 -> 2
- net /LTDC TFT LCD/LTDC_DE: track 0.00 -> 48.8 mm, vias 0 -> 2
- net /LTDC TFT LCD/LTDC_R2: track 0.00 -> 48.3 mm, vias 0 -> 2
- net /LTDC TFT LCD/LTDC_R4: track 0.00 -> 48.2 mm, vias 0 -> 2
- net /MCU/SDIO_CLK: track 0.00 -> 45.4 mm, vias 0 -> 4
- net /MCU/SDIO_D3: track 0.00 -> 44.7 mm, vias 0 -> 2
- net /LTDC TFT LCD/LTDC_G7: track 0.00 -> 42.4 mm
- net /LTDC TFT LCD/LTDC_G1: track 0.00 -> 42.0 mm, vias 0 -> 2
- net /LTDC TFT LCD/LTDC_VSYNC: track 0.00 -> 41.1 mm
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- added copper zone on F.Cu, net Net-(C74-Pad2)
- added copper zone on F.Cu, net Net-(C76-Pad2)
- added copper zone on F.Cu, net Net-(C79-Pad2)
- added copper zone on F.Cu, net Net-(C81-Pad2)
- added copper zone on F.Cu, net Net-(F3-Pad1)
- added copper zone on B.Cu, net VCC
- added copper zone on F.Cu, net VCC
- removed copper zone on F.Cu, net Net-(C29-Pad1)
- removed copper zone on F.Cu, net Net-(C31-Pad2)

Commit message: New SDRAM layout.
Parts:
- added C90: 100nF, Capacitor_SMD:C_0603_1608Metric, B.Cu at (146.7, 103.5)
- moved C11 22.4 mm to (132.8, 105.3), turned to 0 degrees
- moved C59 21.5 mm to (132.8, 108.3), turned to 0 degrees
- moved C47 21.5 mm to (132.8, 104.1), turned to 0 degrees
- moved C50 19.0 mm to (132.6, 106.9)
- moved C43 18.6 mm to (163.9, 99.5), turned to 180 degrees
- moved C46 18.3 mm to (146.7, 101.8), turned to 0 degrees
- moved R23 18.2 mm to (177.6, 113.0)
- moved C44 16.2 mm to (146.7, 93.0), turned to 0 degrees
- moved C45 15.2 mm to (146.7, 82.7), turned to 0 degrees
- moved R22 14.5 mm to (175.0, 113.0)
- moved C61 14.2 mm to (146.7, 97.0), turned to 0 degrees
- moved C38 12.1 mm to (176.3, 113.0), turned to -90 degrees
- moved C42 9.90 mm to (163.9, 94.7)
- moved C2 2.62 mm to (139.5, 100.0), turned to 0 degrees
- moved R18 2.62 mm to (173.3, 113.0), turned to 90 degrees
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Routing:
- net +3.3V: track 361.9 -> 183.2 mm, vias 25 -> 6
- net /LTDC TFT LCD/LTDC_R5: track 53.9 -> 0.00 mm, vias 2 -> 0
- net /LTDC TFT LCD/LTDC_R1: track 53.9 -> 0.00 mm, vias 2 -> 0
- net GND: track 117.6 -> 65.4 mm, vias 19 -> 17
- net /LTDC TFT LCD/LTDC_R0: track 51.9 -> 0.00 mm, vias 2 -> 0
- net /LTDC TFT LCD/LTDC_R6: track 50.9 -> 0.00 mm, vias 2 -> 0
- net /LTDC TFT LCD/LTDC_R3: track 49.8 -> 0.00 mm, vias 2 -> 0
- net /LTDC TFT LCD/LTDC_DE: track 48.8 -> 0.00 mm, vias 2 -> 0
- net /LTDC TFT LCD/LTDC_R2: track 48.3 -> 0.00 mm, vias 2 -> 0
- net /LTDC TFT LCD/LTDC_R4: track 48.2 -> 0.00 mm, vias 2 -> 0
- net /MCU/SDIO_CLK: track 45.4 -> 0.00 mm, vias 4 -> 0
- net /LTDC TFT LCD/LTDC_G7: track 42.4 -> 0.00 mm
- net /LTDC TFT LCD/LTDC_G1: track 42.0 -> 0.00 mm, vias 2 -> 0
- net /MCU/SDIO_D3: track 44.7 -> 2.90 mm, vias 2 -> 0
- net /LTDC TFT LCD/LTDC_VSYNC: track 41.1 -> 0.00 mm
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
Commit message: Finish USB, LoRa Layout
Parts:
- added C100: C_Small, Capacitor_SMD:C_0603_1608Metric, F.Cu at (183.6, 64.5)
- added C101: C_Small, Capacitor_SMD:C_0603_1608Metric, F.Cu at (179.2, 77.2)
- added C102: C_Small, Capacitor_SMD:C_0603_1608Metric, F.Cu at (180.6, 77.2)
- added C103: C_Small, Capacitor_SMD:C_0603_1608Metric, F.Cu at (183.0, 68.1)
- added C104: C_Small, Capacitor_SMD:C_0603_1608Metric, F.Cu at (182.3, 73.4)
- added C105: C_Small, Capacitor_SMD:C_0603_1608Metric, F.Cu at (184.5, 68.1)
- added C106: C_Small, Capacitor_SMD:C_0603_1608Metric, F.Cu at (184.5, 71.1)
- added C107: C_Small, Capacitor_SMD:C_0603_1608Metric, F.Cu at (184.5, 74.2)
- added C108: C_Small, Capacitor_SMD:C_0603_1608Metric, F.Cu at (182.3, 74.9)
- added C109: C_Small, Capacitor_SMD:C_0603_1608Metric, F.Cu at (184.5, 77.2)
- added C110: C_Small, Capacitor_SMD:C_0603_1608Metric, F.Cu at (181.9, 77.2)
- added C111: C_Small, Capacitor_SMD:C_0603_1608Metric, F.Cu at (185.9, 77.2)
- added C112: C_Small, Capacitor_SMD:C_0603_1608Metric, F.Cu at (185.9, 74.2)
- added C113: C_Small, Capacitor_SMD:C_0603_1608Metric, F.Cu at (187.2, 74.2)
- added C114: C_Small, Capacitor_SMD:C_0603_1608Metric, F.Cu at (187.0, 68.9)
- added C115: C_Small, Capacitor_SMD:C_0603_1608Metric, F.Cu at (190.0, 68.1)
- added C116: C_Small, Capacitor_SMD:C_0603_1608Metric, F.Cu at (190.0, 74.2)
- added C117: C_Small, Capacitor_SMD:C_0603_1608Metric, F.Cu at (180.2, 110.0)
- added C91: C_Small, Capacitor_SMD:C_0603_1608Metric, F.Cu at (177.7, 77.2)
- added C92: C_Small, Capacitor_SMD:C_0603_1608Metric, F.Cu at (178.3, 64.5)
- added C93: C_Small, Capacitor_SMD:C_0603_1608Metric, F.Cu at (172.6, 64.5)
- added C94: C_Small, Capacitor_SMD:C_0603_1608Metric, F.Cu at (176.3, 77.2)
- added C95: C_Small, Capacitor_SMD:C_0603_1608Metric, F.Cu at (182.3, 64.5)
- added C96: C_Small, Capacitor_SMD:C_0603_1608Metric, F.Cu at (181.0, 64.5)
- added C97: C_Small, Capacitor_SMD:C_0603_1608Metric, F.Cu at (174.1, 77.2)
- added C98: C_Small, Capacitor_SMD:C_0603_1608Metric, F.Cu at (172.6, 77.2)
- added C99: C_Small, Capacitor_SMD:C_0603_1608Metric, F.Cu at (179.7, 64.5)
- added D11: SS34, Diode_SMD:D_SMA, F.Cu at (188.2, 90.9)
- added D12: SS34, Diode_SMD:D_SMA, F.Cu at (188.2, 103.1)
- added L10: L_Small, Inductor_SMD:L_0603_1608Metric, F.Cu at (183.2, 77.2)
- added L11: L_Small, Inductor_SMD:L_0603_1608Metric, F.Cu at (187.2, 77.2)
- added L12: L_Small, Inductor_SMD:L_0603_1608Metric, F.Cu at (190.0, 71.1)
- added L6: L_Small, Inductor_SMD:L_0603_1608Metric, F.Cu at (180.0, 68.1)
- added L7: L_Small, Inductor_SMD:L_0603_1608Metric, F.Cu at (181.5, 68.1)
- added L8: L_Small, Inductor_SMD:L_0603_1608Metric, F.Cu at (181.5, 71.1)
- added L9: L_Small, Inductor_SMD:L_0603_1608Metric, F.Cu at (183.0, 71.1)
- added Q1: BC847, Package_TO_SOT_SMD:SOT-23, F.Cu at (186.6, 64.8)
- added Q2: BC847, Package_TO_SOT_SMD:SOT-23, F.Cu at (165.4, 114.7)
- added Q3: BC847, Package_TO_SOT_SMD:SOT-23, F.Cu at (168.8, 114.7)
- added R55: R_Small, Resistor_SMD:R_0603_1608Metric, F.Cu at (187.0, 67.4)
- added R56: R_Small, Resistor_SMD:R_0603_1608Metric, F.Cu at (190.0, 65.1)
- added R57: R_Small, Resistor_SMD:R_0603_1608Metric, F.Cu at (188.5, 74.2)
- added R58: R_Small, Resistor_SMD:R_0603_1608Metric, F.Cu at (190.2, 98.3)
- added R59: R_Small, Resistor_SMD:R_0603_1608Metric, F.Cu at (190.2, 93.4)
- added R60: R_Small, Resistor_SMD:R_0603_1608Metric, F.Cu at (185.3, 99.1)
- added R61: R_Small, Resistor_SMD:R_0603_1608Metric, F.Cu at (187.9, 99.1)
- added R62: R_Small, Resistor_SMD:R_0603_1608Metric, F.Cu at (186.6, 99.1)
- added R63: R_Small, Resistor_SMD:R_0603_1608Metric, F.Cu at (191.0, 110.1)
- added R64: R_Small, Resistor_SMD:R_0603_1608Metric, F.Cu at (186.1, 105.9)
- added R65: R_Small, Resistor_SMD:R_0603_1608Metric, F.Cu at (181.5, 110.0)
- added R66: R_Small, Resistor_SMD:R_0603_1608Metric, F.Cu at (189.7, 110.1)
- added R67: R_Small, Resistor_SMD:R_0603_1608Metric, F.Cu at (167.1, 117.5)
- added R68: R_Small, Resistor_SMD:R_0603_1608Metric, F.Cu at (167.1, 112.0)
- added U10: MASWSS0192, Package_TO_SOT_SMD:SOT-363_SC-70-6, F.Cu at (187.0, 71.1)
- added U11: USBLC6-2SC6, Package_TO_SOT_SMD:SOT-23-6, F.Cu at (188.7, 95.8)
- added U12: USBLC6-2SC6, Package_TO_SOT_SMD:SOT-23-6, F.Cu at (189.7, 106.8)
- added Y4: 32MHz, Crystal:Crystal_SMD_3225-4Pin_3.2x2.5mm, F.Cu at (175.4, 64.5)
- J4: value xAnt2 -> SWD_LOG; footprint Anh_Footprints:Connector_Coaxial_SMA -> Connector_PinHeader_2.54mm:PinHeader_2x03_P2.54mm_Horizontal
- J9: value xAnt1 -> LoRa_Anten
- U6: value Ai-Thinker-Ra-02 -> SX1278; footprint RF_Module:Ai-Thinker-Ra-01-LoRa -> Package_DFN_QFN:QFN-28-1EP_6x6mm_P0.65mm_EP4.8x4.8mm
- U9: value CP2102N-Axx-xQFN28 -> CP2102N
- moved U6 114.2 mm to (175.4, 71.5), turned to -90 degrees
- moved C49 32.3 mm to (139.5, 90.8)
- moved J4 9.23 mm to (187.8, 80.8), turned to 0 degrees
- moved C16 6.76 mm to (139.5, 84.0)
- moved C15 3.90 mm to (171.5, 84.4), turned to 180 degrees
- moved R3 2.59 mm to (171.5, 88.3)
- moved JP3 2.08 mm to (173.8, 87.2)
- moved U9 1.93 mm to (185.7, 111.7), turned to -90 degrees
- moved J10 1.59 mm to (197.1, 94.5)
- moved C54 1.38 mm to (156.9, 109.0), turned to 90 degrees
- moved C60 1.23 mm to (171.5, 90.9)
- moved J11 1.14 mm to (197.1, 106.7)
- moved R5 1.06 mm to (159.5, 109.0)
- moved R12 1.04 mm to (158.2, 109.0)
- moved C51 1.03 mm to (171.5, 95.8), turned to 180 degrees
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Connections:
- net /WIFI ESP32/ETH_REFCLK renamed /USB/WiFi_BOOT
- net Net-(C25-Pad2) renamed /USB/WiFi_RST
- J10 pad A1: Net-(J10-PadA1) -> GND
- J10 pad A12: Net-(J10-PadA1) -> GND
- J10 pad A5: unconnected-(J10-PadA5) -> Net-(J10-PadA5)
- J10 pad A6: unconnected-(J10-PadA6) -> Net-(J10-PadA6)
- J10 pad A7: unconnected-(J10-PadA7) -> Net-(J10-PadA7)
- J10 pad B1: Net-(J10-PadA1) -> GND
- J10 pad B12: Net-(J10-PadA1) -> GND
- J10 pad B5: unconnected-(J10-PadB5) -> Net-(J10-PadB5)
- J10 pad B6: unconnected-(J10-PadB6) -> Net-(J10-PadA6)
- J10 pad B7: unconnected-(J10-PadB7) -> Net-(J10-PadA7)
- J10 pad S1: unconnected-(J10-PadS1) -> GND
- J11 pad A1: Net-(J11-PadA1) -> GND
- J11 pad A12: Net-(J11-PadA1) -> GND
- J11 pad A5: unconnected-(J11-PadA5) -> Net-(J11-PadA5)
- J11 pad A6: unconnected-(J11-PadA6) -> Net-(J11-PadA6)
- J11 pad A7: unconnected-(J11-PadA7) -> Net-(J11-PadA7)
- J11 pad B1: Net-(J11-PadA1) -> GND
- J11 pad B12: Net-(J11-PadA1) -> GND
- J11 pad B5: unconnected-(J11-PadB5) -> Net-(J11-PadB5)
- J11 pad B6: unconnected-(J11-PadB6) -> Net-(J11-PadA6)
- J11 pad B7: unconnected-(J11-PadB7) -> Net-(J11-PadA7)
- J11 pad S1: unconnected-(J11-PadS1) -> GND
- J4 pad 1: unconnected-(J4-Pad1) -> +3.3V
- J4 pad 2: GND -> LOG_TX
- J9 pad 1: unconnected-(J9-Pad1) -> Net-(C116-Pad2)
- U4 pad 40: /WIFI ESP32/ESP_FLASH_RX -> /USB/TXD
- U4 pad 41: /WIFI ESP32/ESP_FLASH_TX -> /USB/RXD
- U6 pad 1: Net-(U6-Pad1) -> Net-(L6-Pad1)
- U6 pad 14: unconnected-(U6-Pad14) -> +3.3V
- U6 pad 15: unconnected-(U6-Pad15) -> GND
- U6 pad 16: Net-(U6-Pad1) -> /RF-LORA-ZIGBEE/LoRa_SCK
- U6 pad 2: Net-(U6-Pad1) -> Net-(C100-Pad1)
- U6 pad 3: unconnected-(U6-Pad3) -> +3.3V
- U6 pad 4: unconnected-(U6-Pad4) -> Net-(C99-Pad1)
- U6 pad 5: unconnected-(U6-Pad5) -> Net-(C92-Pad2)
- U6 pad 6: unconnected-(U6-Pad6) -> Net-(C93-Pad2)
- U6 pad 7: unconnected-(U6-Pad7) -> /RF-LORA-ZIGBEE/LoRa_RST
- U6 pad 8: unconnected-(U6-Pad8) -> /RF-LORA-ZIGBEE/LoRa_IRQ
- U6 pad 9: Net-(U6-Pad1) -> unconnected-(U6-Pad9)
- U9 pad 24: unconnected-(U9-Pad24) -> Net-(Q3-Pad2)
- U9 pad 25: unconnected-(U9-Pad25) -> /USB/RXD
- U9 pad 26: unconnected-(U9-Pad26) -> Net-(R66-Pad2)
- U9 pad 28: unconnected-(U9-Pad28) -> Net-(Q2-Pad2)
- U9 pad 29: Net-(U9-Pad29) -> GND
- U9 pad 3: Net-(U9-Pad29) -> GND
- U9 pad 4: unconnected-(U9-Pad4) -> Net-(J11-PadA6)
- U9 pad 5: unconnected-(U9-Pad5) -> Net-(J11-PadA7)
- U9 pad 6: unconnected-(U9-Pad6) -> Net-(C117-Pad1)
- U9 pad 7: unconnected-(U9-Pad7) -> +5V
- U9 pad 8: unconnected-(U9-Pad8) -> +5V
- U9 pad 9: unconnected-(U9-Pad9) -> Net-(R65-Pad1)
Routing:
- net +3.3V: track 183.2 -> 245.9 mm, vias 6 -> 8
- net /LTDC TFT LCD/LTDC_R1: track 0.00 -> 50.7 mm, vias 0 -> 2
- net /LTDC TFT LCD/LTDC_R5: track 0.00 -> 50.1 mm, vias 0 -> 2
- net /LTDC TFT LCD/LTDC_R0: track 0.00 -> 48.5 mm, vias 0 -> 2
- net GND: track 65.4 -> 113.8 mm, vias 17 -> 23
- net /LTDC TFT LCD/LTDC_R3: track 0.00 -> 48.0 mm, vias 0 -> 2
- net /LTDC TFT LCD/LTDC_R2: track 0.00 -> 47.2 mm, vias 0 -> 2
- net /LTDC TFT LCD/LTDC_R6: track 0.00 -> 46.9 mm, vias 0 -> 2
- net /LTDC TFT LCD/LTDC_R4: track 0.00 -> 46.6 mm, vias 0 -> 2
- net /LTDC TFT LCD/LTDC_R7: track 0.00 -> 43.7 mm, vias 0 -> 2
- net /LTDC TFT LCD/LTDC_DE: track 0.00 -> 36.7 mm, vias 0 -> 2
- net /LTDC TFT LCD/LTDC_G1: track 0.00 -> 31.0 mm, vias 0 -> 2
- net /LTDC TFT LCD/LTDC_VSYNC: track 0.00 -> 30.6 mm
- net /LTDC TFT LCD/LTDC_G3: track 0.00 -> 30.2 mm
- net /LTDC TFT LCD/LTDC_HSYNC: track 0.00 -> 29.1 mm
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
Commit message: Finish LTDC LCD Layout
Parts:
- moved R68 5.58 mm to (165.4, 117.3)
- moved R67 1.73 mm to (168.8, 117.3)
- moved Q2 0.16 mm to (165.4, 114.6)
- moved Q3 0.16 mm to (168.8, 114.6)
Routing:
- net SWDIO: track 0.00 -> 55.0 mm, vias 0 -> 1
- net SWCLK: track 0.00 -> 50.8 mm, vias 0 -> 1
- net /MCU/SDIO_CLK: track 0.00 -> 47.6 mm, vias 0 -> 2
- net /LTDC TFT LCD/LTDC_PCLK: track 0.00 -> 47.5 mm, vias 0 -> 2
- net /MCU/SDIO_CMD: track 2.63 -> 48.7 mm, vias 0 -> 2
- net /MCU/USB_OTG_DM: track 0.00 -> 41.9 mm, vias 0 -> 2
- net /MCU/SDIO_D3: track 2.82 -> 43.5 mm, vias 0 -> 2
- net /MCU/USB_OTG_DP: track 0.00 -> 39.7 mm, vias 0 -> 2
- net /MCU/SDIO_D2: track 2.68 -> 41.2 mm, vias 0 -> 2
- net /LTDC TFT LCD/LTDC_B2: track 14.1 -> 45.3 mm, vias 0 -> 2
- net /LTDC TFT LCD/LTDC_B4: track 19.2 -> 49.5 mm
- net /LTDC TFT LCD/LTDC_B3: track 16.4 -> 46.7 mm, vias 0 -> 2
- net /LTDC TFT LCD/LTDC_B7: track 21.2 -> 51.4 mm
- net /LTDC TFT LCD/LTDC_B6: track 19.0 -> 48.9 mm
- net /LTDC TFT LCD/LTDC_B5: track 21.4 -> 51.1 mm
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