File: GatewayPlus_V1.1.kicad_pcb (KiCad board)
At the start: 2 copper layers, 100 x 67 mm, 267 parts, among them IC1 MP1584EN, IC2 MP1584EN, J1 LTDC_LCD_FPC_40p, J10 USB_OTG, J11 USB_WIFI_FLASH, J2 Micro_SD_Card, J3 ESP Anten, J4 SWD_LOG, J5 HR911105A, J6 RS485, J7 Conn_Jack-DC, J8 AudioJack4, J9 LoRa_Anten, Q1 BC847, Q2 BC847, Q3 BC847, SW1 SW_Push, SW2 ESP_RESET, SW3 ESP_BOOT, U1 STM32F429IGTx, U10 MASWSS0192, U11 USBLC6-2SC6, U12 USBLC6-2SC6, U2 IS42S16400J - HY57V641620E, U3 W25Q128JVS, U4 ESP32-D0WD-V3, U5 W25Q32JVSS, U6 SX1278, U7 LAN8720A, U8 MAX485E, U9 CP2102N, X1 50MHz, Y1 32.768KHz, Y2 25MHz, Y3 40MHz, Y4 32MHz

Commit message: .
Parts:
- added C118: 10uF, Capacitor_SMD:C_1206_3216Metric, F.Cu at (184.0, 80.8)
- moved C59 20.8 mm to (153.6, 109.0), turned to 90 degrees
- moved C50 16.3 mm to (139.5, 92.1)
- moved C41 10.8 mm to (133.0, 97.6)
- moved R41 10.7 mm to (122.3, 99.1), turned to 180 degrees
- moved C47 9.40 mm to (139.5, 97.5)
- moved C11 7.22 mm to (139.5, 102.6)
- moved C71 1.31 mm to (133.0, 98.9)
- moved R10 0.45 mm to (185.0, 84.1)
- moved C72 0.43 mm to (130.0, 98.3)
- moved J4 0.36 mm to (188.1, 80.8)
- moved C14 0.36 mm to (139.5, 96.2)
- moved C19 0.34 mm to (145.3, 109.0)
- turned R34 to 0 degrees
- turned R35 to 0 degrees
Routing:
- net +3.3V: track 261.9 -> 386.1 mm, vias 8 -> 15
- net +5V: track 4.44 -> 39.2 mm, vias 1 -> 2
- net GND: track 113.8 -> 137.7 mm, vias 23 -> 58
- net Net-(D5-Pad1): track 0.00 -> 22.6 mm
- net Net-(D6-Pad1): track 0.00 -> 17.4 mm, vias 0 -> 2
- net Net-(C1-Pad2): track 6.55 -> 20.0 mm, vias 0 -> 2
- net /RS485/A+: track 0.00 -> 11.5 mm
- net /RS485/B-: track 0.00 -> 9.92 mm
- net Net-(C29-Pad1): track 1.48 -> 7.09 mm
- net Net-(J1-Pad1): track 0.00 -> 3.99 mm
- net Net-(R36-Pad2): track 0.00 -> 3.28 mm
- net Net-(R37-Pad2): track 0.00 -> 3.23 mm
- net Net-(D12-Pad2): track 7.62 -> 10.7 mm
- net /MCU/SDRAM_D4: track 23.3 -> 20.3 mm, vias 1 -> 3
- net /MCU/USART2_TX: track 0.00 -> 2.56 mm, vias 0 -> 1
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- added copper zone on F.Cu, net Net-(C29-Pad1)
- added copper zone on F.Cu, net Net-(C31-Pad2)
