File: GatewayPlus_V1.1.kicad_sch (KiCad schematic)
At the start: 14 parts

Commit message: Finish USB, LoRa Layout
Connections:
- net WIFI ESP32/ETH_REFCLK renamed USB/WiFi_BOOT
Other:
- sheet RF-LORA-ZIGBEE ports: added LoRa_IRQ, LoRa_MISO, LoRa_MOSI, LoRa_NSS, LoRa_RST, LoRa_SCK; removed none
- sheet USB ports: added OTG_DM, OTG_DP, RXD, TXD, WiFi_BOOT, WiFi_RST; removed none
- sheet WIFI ESP32 ports: added WiFi_RST; removed none

Commit message: .
Other:
- sheet MCU ports: added LoRa_CS, LoRa_IRQ, LoRa_RST, SPI5_MISO, SPI5_MOSI, SPI5_SCK, USART6_RX, USART6_TX; removed USART2_RX, USART2_TX
Changed lines of the file:
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@@
+    (stroke (width 0) (type default) (color 0 0 0 0))
+  )
+  (wire (pts (xy 144.78 77.47) (xy 165.1 77.47))
     (stroke (width 0) (type default) (color 0 0 0 0))
   )
@@
     (stroke (width 0) (type default) (color 0 0 0 0))
   )
+  (wire (pts (xy 144.78 80.01) (xy 165.1 80.01))
+    (stroke (width 0) (type default) (color 0 0 0 0))
+  )
   (wire (pts (xy 200.66 184.15) (xy 200.66 198.12))
     (stroke (width 0) (type default) (color 0 0 0 0))
@@
     (stroke (width 0) (type default) (color 0 0 0 0))
   )
+  (wire (pts (xy 144.78 82.55) (xy 165.1 82.55))
+    (stroke (width 0) (type default) (color 0 0 0 0))
+  )
   (wire (pts (xy 248.92 121.92) (xy 308.61 121.92))
     (stroke (width 0) (type default) (color 0 0 0 0))
@@
     (stroke (width 0) (type default) (color 0 0 0 0))
   )
+  (wire (pts (xy 144.78 71.12) (xy 165.1 71.12))
+    (stroke (width 0) (type default) (color 0 0 0 0))
+  )
   (wire (pts (xy 144.78 102.87) (xy 165.1 102.87))
     (stroke (width 0) (type default) (color 0 0 0 0))
@@
     (stroke (width 0) (type default) (color 0 0 0 0))
   )
+  (wire (pts (xy 144.78 85.09) (xy 165.1 85.09))
+    (stroke (width 0) (type default) (color 0 0 0 0))
+  )
   (wire (pts (xy 259.08 171.45) (xy 259.08 130.81))
     (stroke (width 0) (type default) (color 0 0 0 0))
@@
   )
   (wire (pts (xy 184.15 195.58) (xy 181.61 195.58))
+    (stroke (width 0) (type default) (color 0 0 0 0))
+  )
+  (wire (pts (xy 144.78 68.58) (xy 165.1 68.58))
     (stroke (width 0) (type default) (color 0 0 0 0))
   )
@@
     )
   )
-  (sheet (at 165.1 59.69) (size 57.15 124.46) (fields_autoplaced)
+  (sheet (at 165.1 64.77) (size 57.15 119.38) (fields_autoplaced)
     (stroke (width 0.1524) (type solid) (color 0 0 0 0))
     (fill (color 0 0 0 0.0000))
-    (property "Sheet name" "MCU" (id 0) (at 165.1 58.9784 0)
+    (property "Sheet name" "MCU" (id 0) (at 165.1 64.0584 0)
       (effects (font (size 1.27 1.27)) (justify left bottom))
     )
@@
       (effects (font (size 1.27 1.27)) (justify left))
     )
-    (pin "SPI1_SCK" bidirectional (at 165.1 179.07 180)
-      (effects (font (size 1.27 1.27)) (justify left))
-    )
-    (pin "SPI1_MISO" bidirectional (at 165.1 173.99 180)
-      (effects (font (size 1.27 1.27)) (justify left))
-    )
-    (pin "SPI1_MOSI" bidirectional (at 165.1 176.53 180)
+    (pin "SPI5_SCK" bidirectional (at 165.1 179.07 180)
+      (effects (font (size 1.27 1.27)) (justify left))
+    )
+    (pin "SPI5_MISO" bidirectional (at 165.1 173.99 180)
+      (effects (font (size 1.27 1.27)) (justify left))
+    )
+    (pin "SPI5_MOSI" bidirectional (at 165.1 176.53 180)
       (effects (font (size 1.27 1.27)) (justify left))
     )
@@
       (effects (font (size 1.27 1.27)) (justify right))
     )
-    (pin "USART2_RX" bidirectional (at 184.15 184.15 270)
-      (effects (font (size 1.27 1.27)) (justify left))
-    )
-    (pin "USART2_TX" bidirectional (at 189.23 184.15 270)
+    (pin "USART6_RX" bidirectional (at 184.15 184.15 270)
+      (effects (font (size 1.27 1.27)) (justify left))
+    )
+    (pin "USART6_TX" bidirectional (at 189.23 184.15 270)
       (effects (font (size 1.27 1.27)) (justify left))
     )
     (pin "RS485_TE" bidirectional (at 186.69 184.15 270)
+      (effects (font (size 1.27 1.27)) (justify left))
+    )
+    (pin "LoRa_IRQ" bidirectional (at 165.1 68.58 180)
+      (effects (font (size 1.27 1.27)) (justify left))
+    )
+    (pin "LoRa_CS" bidirectional (at 165.1 77.47 180)
+      (effects (font (size 1.27 1.27)) (justify left))
+    )
+    (pin "LoRa_RST" bidirectional (at 165.1 71.12 180)
+      (effects (font (size 1.27 1.27)) (justify left))
+    )
+    (pin "SPI1_MISO" bidirectional (at 165.1 82.55 180)
+      (effects (font (size 1.27 1.27)) (justify left))
+    )
+    (pin "SPI1_MOSI" bidirectional (at 165.1 85.09 180)
+      (effects (font (size 1.27 1.27)) (justify left))
+    )
+    (pin "SPI1_SCK" bidirectional (at 165.1 80.01 180)
       (effects (font (size 1.27 1.27)) (justify left))
     )
@@
     )
   )
-  (sheet (at 115.57 59.69) (size 29.21 29.21) (fields_autoplaced)
+  (sheet (at 115.57 64.77) (size 29.21 24.13) (fields_autoplaced)
     (stroke (width 0.1524) (type solid) (color 0 0 0 0))
     (fill (color 0 0 0 0.0000))
-    (property "Sheet name" "RF-LORA-ZIGBEE" (id 0) (at 115.57 58.9784 0)
+    (property "Sheet name" "RF-LORA-ZIGBEE" (id 0) (at 115.57 64.0584 0)
       (effects (font (size 1.27 1.27)) (justify left bottom))
     )
@@
       (effects (font (size 1.27 1.27)) (justify left top))
     )
-    (pin "LoRa_IRQ" bidirectional (at 144.78 71.12 0)
-      (effects (font (size 1.27 1.27)) (justify right))
-    )
-    (pin "LoRa_SCK" bidirectional (at 144.78 78.74 0)
-      (effects (font (size 1.27 1.27)) (justify right))
-    )
-    (pin "LoRa_RST" bidirectional (at 144.78 73.66 0)
-      (effects (font (size 1.27 1.27)) (justify right))
-    )
-    (pin "LoRa_MISO" bidirectional (at 144.78 81.28 0)
-      (effects (font (size 1.27 1.27)) (justify right))
-    )
-    (pin "LoRa_MOSI" bidirectional (at 144.78 83.82 0)
-      (effects (font (size 1.27 1.27)) (justify right))
-    )
-    (pin "LoRa_NSS" bidirectional (at 144.78 86.36 0)
-      (effects (font (size 1.27 1.27)) (justify right))
-    )
-  )
-  (sheet (at 308.61 59.69) (size 29.21 15.24) (fields_autoplaced)
+    (pin "LoRa_IRQ" bidirectional (at 144.78 68.58 0)
+      (effects (font (size 1.27 1.27)) (justify right))
+    )
+    (pin "LoRa_SCK" bidirectional (at 144.78 80.01 0)
+      (effects (font (size 1.27 1.27)) (justify right))
+    )
+    (pin "LoRa_RST" bidirectional (at 144.78 71.12 0)
+      (effects (font (size 1.27 1.27)) (justify right))
+    )
+    (pin "LoRa_MISO" bidirectional (at 144.78 82.55 0)
+      (effects (font (size 1.27 1.27)) (justify right))
+    )
+    (pin "LoRa_MOSI" bidirectional (at 144.78 85.09 0)
+      (effects (font (size 1.27 1.27)) (justify right))
+    )
+    (pin "LoRa_NSS" bidirectional (at 144.78 77.47 0)
+      (effects (font (size 1.27 1.27)) (justify right))
+    )
+  )
+  (sheet (at 308.61 64.77) (size 29.21 15.24) (fields_autoplaced)
     (stroke (width 0.1524) (type solid) (color 0 0 0 0))
     (fill (color 0 0 0 0.0000))
-    (property "Sheet name" "AUDIO" (id 0) (at 308.61 58.9784 0)
+    (property "Sheet name" "AUDIO" (id 0) (at 308.61 64.0584 0)
       (effects (font (size 1.27 1.27)) (justify left bottom))
     )
-    (property "Sheet file" "AUDIO.kicad_sch" (id 1) (at 308.61 75.5146 0)
+    (property "Sheet file" "AUDIO.kicad_sch" (id 1) (at 308.61 80.5946 0)
       (effects (font (size 1.27 1.27)) (justify left top))
     )
@@
       (reference "R68") (unit 1) (value "R_Small") (footprint "Resistor_SMD:R_0603_1608Metric")
     )
+    (path "/77c5f343-dce2-4f5b-a810-1e60994fab1d/8ebb2caa-7a65-42c6-ad22-d411d76c7e44"
+      (reference "R69") (unit 1) (value "R_Small") (footprint "Resistor_SMD:R_0603_1608Metric")
+    )
+    (path "/77c5f343-dce2-4f5b-a810-1e60994fab1d/2be6c116-d1ab-4da5-ae65-6266b8b0934c"
+      (reference "R70") (unit 1) (value "R_Small") (footprint "Resistor_SMD:R_0603_1608Metric")
+    )
     (path "/4931c4f2-ec98-49ed-98f1-a79587b46d92/80468874-9f96-44a2-871d-c1b88eec0daf"

Commit message: Create Audio CODEC schematic block and layout.
Other:
- sheet AUDIO ports: added LRCLK, MCLK, SCL, SCLK, SDA, SDIN, SDOUT; removed none

Commit message: Only 1 wire to complete.
Other:
- sheet MCU ports: added I2C2_SCL, I2C2_SDA, I2S2_DIN, I2S2_DOUT, I2S2_SCK, I2S2_WS, MCO_MCLK; removed none
