File: MCU.kicad_sch (KiCad schematic)
At the start: 46 parts, among them SW1 SW_Push, U1 STM32F429IGTx, Y1 32.768KHz, Y2 25MHz

Commit message: Finish USB, LoRa Layout
Parts:
- added J4: SWD_LOG, Connector_PinHeader_2.54mm:PinHeader_2x03_P2.54mm_Horizontal, symbol Connector_Generic:Conn_02x03_Odd_Even
Connections:
- net +3.3V: now also J4.1 (Pin_1)
- net GND: now also J4.6 (Pin_6)
- net SWCLK: now also J4.5 (Pin_5)
- net SWDIO: now also J4.3 (Pin_3)
- new net LOG_RX: J4.4 (Pin_4)
- new net LOG_TX: J4.2 (Pin_2)
Other:
- moved on the sheet: C6, C7, C8, C9, D1, R6, R7, Y1, Y2

Commit message: .
Parts:
- added C118: 10uF, Capacitor_SMD:C_1206_3216Metric, symbol Device:C_Small
Connections:
- net +3.3V: now also C118.2
- net GND: now also C118.1
Changed lines of the file:
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@@
     (pin "2")
+  )
+  (symbol (lib_id "Device:C_Small") (at 201.93 168.91 180) (unit 1)
+    (in_bom yes) (on_board yes)
+    (property "Reference" "C118" (id 0) (at 200.66 171.45 90))
+    (property "Value" "10uF" (id 1) (at 200.66 163.83 90))
+    (property "Footprint" "Capacitor_SMD:C_1206_3216Metric" (id 2) (at 201.93 168.91 0)
+      (effects (font (size 1.27 1.27)) hide)
+    )
+    (property "Datasheet" "~" (id 3) (at 201.93 168.91 0)
+      (effects (font (size 1.27 1.27)) hide)
+    )
+    (pin "1")
+    (pin "2")
+  )
+  (symbol (lib_id "power:+3.3V") (at 201.93 166.37 0) (mirror y) (unit 1)
+    (in_bom yes) (on_board yes) (fields_autoplaced)
+    (property "Reference" "#PWR0253" (id 0) (at 201.93 170.18 0)
+      (effects (font (size 1.27 1.27)) hide)
+    )
+    (property "Value" "+3.3V" (id 1) (at 201.93 161.29 0))
+    (property "Footprint" "" (id 2) (at 201.93 166.37 0)
+      (effects (font (size 1.27 1.27)) hide)
+    )
+    (property "Datasheet" "" (id 3) (at 201.93 166.37 0)
+      (effects (font (size 1.27 1.27)) hide)
+    )
+    (pin "1")
   )
   (symbol (lib_id "Device:C_Small") (at 238.76 107.95 270) (mirror x) (unit 1)
@@
     (pin "99")
   )
+  (symbol (lib_id "power:GND") (at 201.93 171.45 0) (mirror y) (unit 1)
+    (in_bom yes) (on_board yes) (fields_autoplaced)
+    (property "Reference" "#PWR0252" (id 0) (at 201.93 177.8 0)
+      (effects (font (size 1.27 1.27)) hide)
+    )
+    (property "Value" "GND" (id 1) (at 201.93 176.53 0))
+    (property "Footprint" "" (id 2) (at 201.93 171.45 0)
+      (effects (font (size 1.27 1.27)) hide)
+    )
+    (property "Datasheet" "" (id 3) (at 201.93 171.45 0)
+      (effects (font (size 1.27 1.27)) hide)
+    )
+    (pin "1")
+  )
 )

Commit message: .
Parts:
- added R69, R70: R_Small, Resistor_SMD:R_0603_1608Metric, symbol Device:R_Small
Connections:
- net LOG_TX is gone; now on net GND: J4.2 (Pin_2)
- net GND: no longer J4.6 (Pin_6)
- net SPI1_MISO: now also U1.162 (PB4); no longer U1.26 (PF8)
- net SPI1_MOSI: now also U1.163 (PB5); no longer U1.27 (PF9)
- net SPI1_SCK: now also U1.161 (PB3); no longer U1.25 (PF7)
- net USART2_RX: now also R70.2
- net USART2_TX: now also R69.2
- net LoRa_CS: now reaches U1.1 (PE2)
- net USART6_TX: now reaches U1.115 (PC6)
- net USART6_RX: now reaches U1.116 (PC7)
- net LoRa_RST: now reaches U1.2 (PE3)
- net LoRa_IRQ: now reaches U1.40 (PA0)
- net LOG_RX: no longer names the net of J4.4 (Pin_4)
- net LOG_RX: now also R69.1
- new net: J4.6 (Pin_6), R70.1
- new net SPI5_MISO: U1.26 (PF8)
- new net SPI5_MOSI: U1.27 (PF9)
- new net SPI5_SCK: U1.25 (PF7)
Changed lines of the file:
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@@
+    )
+  )
+  (global_label "USART2_TX" (shape bidirectional) (at 144.78 238.76 0) (fields_autoplaced)
+    (effects (font (size 1.27 1.27)) (justify left))
+    (property "Intersheet References" "${INTERSHEET_REFS}" (id 0) (at 157.4136 238.6806 0)
+      (effects (font (size 1.27 1.27)) (justify left) hide)
     )
   )
@@
     )
   )
+  (global_label "USART2_RX" (shape bidirectional) (at 234.95 171.45 0) (fields_autoplaced)
+    (effects (font (size 1.27 1.27)) (justify left))
+    (property "Intersheet References" "${INTERSHEET_REFS}" (id 0) (at 247.886 171.3706 0)
+      (effects (font (size 1.27 1.27)) (justify left) hide)
+    )
+  )
   (global_label "LSEI" (shape bidirectional) (at 144.78 218.44 0) (fields_autoplaced)
     (effects (font (size 1.27 1.27)) (justify left))
@@
     )
   )
-  (global_label "LOG_TX" (shape bidirectional) (at 229.87 166.37 0) (fields_autoplaced)
-    (effects (font (size 1.27 1.27)) (justify left))
-    (property "Intersheet References" "${INTERSHEET_REFS}" (id 0) (at 239.0564 166.2906 0)
-      (effects (font (size 1.27 1.27)) (justify left) hide)
-    )
-  )
   (global_label "SWDIO" (shape bidirectional) (at 217.17 168.91 180) (fields_autoplaced)
     (effects (font (size 1.27 1.27)) (justify right))
@@
     )
   )
-  (global_label "LOG_RX" (shape bidirectional) (at 229.87 168.91 0) (fields_autoplaced)
-    (effects (font (size 1.27 1.27)) (justify left))
-    (property "Intersheet References" "${INTERSHEET_REFS}" (id 0) (at 239.3588 168.8306 0)
-      (effects (font (size 1.27 1.27)) (justify left) hide)
-    )
-  )
   (global_label "HSEI" (shape bidirectional) (at 226.06 127 180) (fields_autoplaced)
     (effects (font (size 1.27 1.27)) (justify right))
@@
     )
   )
+  (global_label "USART2_RX" (shape bidirectional) (at 144.78 241.3 0) (fields_autoplaced)
+    (effects (font (size 1.27 1.27)) (justify left))
+    (property "Intersheet References" "${INTERSHEET_REFS}" (id 0) (at 157.716 241.2206 0)
+      (effects (font (size 1.27 1.27)) (justify left) hide)
+    )
+  )
   (global_label "LSEI" (shape bidirectional) (at 226.06 115.57 180) (fields_autoplaced)
     (effects (font (size 1.27 1.27)) (justify right))
@@
     )
   )
+  (global_label "USART2_TX" (shape bidirectional) (at 234.95 168.91 0) (fields_autoplaced)
+    (effects (font (size 1.27 1.27)) (justify left))
+    (property "Intersheet References" "${INTERSHEET_REFS}" (id 0) (at 247.5836 168.8306 0)
+      (effects (font (size 1.27 1.27)) (justify left) hide)
+    )
+  )
   (global_label "STATUS LED" (shape bidirectional) (at 144.78 215.9 0) (fields_autoplaced)
     (effects (font (size 1.27 1.27)) (justify left))
@@
     (effects (font (size 1.27 1.27)) (justify right))
   )
-  (hierarchical_label "USART2_TX" (shape bidirectional) (at 144.78 238.76 0)
-    (effects (font (size 1.27 1.27)) (justify left))
-  )
   (hierarchical_label "SDRAM_NBL0" (shape bidirectional) (at 144.78 269.24 0)
     (effects (font (size 1.27 1.27)) (justify left))
@@
     (effects (font (size 1.27 1.27)) (justify left))
   )
-  (hierarchical_label "SPI1_MISO" (shape bidirectional) (at 71.12 289.56 180)
+  (hierarchical_label "SPI5_MISO" (shape bidirectional) (at 71.12 289.56 180)
     (effects (font (size 1.27 1.27)) (justify right))
   )
@@
     (effects (font (size 1.27 1.27)) (justify left))
   )
+  (hierarchical_label "SPI1_MOSI" (shape bidirectional) (at 144.78 152.4 0)
+    (effects (font (size 1.27 1.27)) (justify left))
+  )
   (hierarchical_label "LTDC_G[0..7]" (shape bidirectional) (at 170.18 284.48 0)
     (effects (font (size 1.27 1.27)) (justify left))
   )
+  (hierarchical_label "LoRa_CS" (shape bidirectional) (at 144.78 274.32 0)
+    (effects (font (size 1.27 1.27)) (justify left))
+  )
   (hierarchical_label "SDIO_CMD" (shape bidirectional) (at 144.78 231.14 0)
     (effects (font (size 1.27 1.27)) (justify left))
@@
     (effects (font (size 1.27 1.27)) (justify left))
   )
+  (hierarchical_label "LoRa_RST" (shape bidirectional) (at 144.78 276.86 0)
+    (effects (font (size 1.27 1.27)) (justify left))
+  )
   (hierarchical_label "SDRAM_A[0..11]" (shape bidirectional) (at 50.8 228.6 180)
     (effects (font (size 1.27 1.27)) (justify right))
@@
     (effects (font (size 1.27 1.27)) (justify right))
   )
-  (hierarchical_label "USART2_RX" (shape bidirectional) (at 144.78 241.3 0)
-    (effects (font (size 1.27 1.27)) (justify left))
-  )
   (hierarchical_label "LTDC_R[0..7]" (shape bidirectional) (at 40.64 243.84 180)
     (effects (font (size 1.27 1.27)) (justify right))
   )
+  (hierarchical_label "USART6_TX" (shape bidirectional) (at 144.78 198.12 0)
+    (effects (font (size 1.27 1.27)) (justify left))
+  )
   (hierarchical_label "USART1_RX" (shape bidirectional) (at 144.78 121.92 0)
     (effects (font (size 1.27 1.27)) (justify left))
   )
+  (hierarchical_label "USART6_RX" (shape bidirectional) (at 144.78 200.66 0)
+    (effects (font (size 1.27 1.27)) (justify left))
+  )
   (hierarchical_label "I2C1_SDA" (shape bidirectional) (at 144.78 162.56 0)
     (effects (font (size 1.27 1.27)) (justify left))
@@
     (effects (font (size 1.27 1.27)) (justify left))
   )
+  (hierarchical_label "SPI1_MISO" (shape bidirectional) (at 144.78 149.86 0)
+    (effects (font (size 1.27 1.27)) (justify left))
+  )
   (hierarchical_label "RMII_TXD0" (shape bidirectional) (at 144.78 170.18 0)
     (effects (font (size 1.27 1.27)) (justify left))
   )
+  (hierarchical_label "LoRa_IRQ" (shape bidirectional) (at 144.78 96.52 0)
+    (effects (font (size 1.27 1.27)) (justify left))
+  )
   (hierarchical_label "SDRAM_NWE" (shape bidirectional) (at 144.78 182.88 0)
     (effects (font (size 1.27 1.27)) (justify left))
@@
     (effects (font (size 1.27 1.27)) (justify left))
   )
-  (hierarchical_label "SPI1_MOSI" (shape bidirectional) (at 71.12 292.1 180)
+  (hierarchical_label "SPI5_MOSI" (shape bidirectional) (at 71.12 292.1 180)
     (effects (font (size 1.27 1.27)) (justify right))
   )
@@
     (effects (font (size 1.27 1.27)) (justify left))
   )
-  (hierarchical_label "SPI1_SCK" (shape bidirectional) (at 71.12 287.02 180)
+  (hierarchical_label "SPI1_SCK" (shape bidirectional) (at 144.78 147.32 0)
+    (effects (font (size 1.27 1.27)) (justify left))
+  )
+  (hierarchical_label "SPI5_SCK" (shape bidirectional) (at 71.12 287.02 180)
     (effects (font (size 1.27 1.27)) (justify right))
   )
@@
     (pin "2")
   )
+  (symbol (lib_id "Device:R_Small") (at 232.41 171.45 90) (unit 1)
+    (in_bom yes) (on_board yes)
+    (property "Reference" "R70" (id 0) (at 232.41 168.91 90))
+    (property "Value" "R_Small" (id 1) (at 232.41 173.99 90))
+    (property "Footprint" "Resistor_SMD:R_0603_1608Metric" (id 2) (at 232.41 171.45 0)
+      (effects (font (size 1.27 1.27)) hide)
+    )
+    (property "Datasheet" "~" (id 3) (at 232.41 171.45 0)
+      (effects (font (size 1.27 1.27)) hide)
+    )
+    (pin "1")
+    (pin "2")
+  )
   (symbol (lib_id "power:+3.3V") (at 213.36 52.07 0) (mirror y) (unit 1)
     (in_bom yes) (on_board yes) (fields_autoplaced)
@@
     )
     (pin "1")
+  )
+  (symbol (lib_id "Device:R_Small") (at 232.41 168.91 90) (unit 1)
+    (in_bom yes) (on_board yes)
+    (property "Reference" "R69" (id 0) (at 232.41 166.37 90))
+    (property "Value" "R_Small" (id 1) (at 232.41 171.45 90))
+    (property "Footprint" "Resistor_SMD:R_0603_1608Metric" (id 2) (at 232.41 168.91 0)
+      (effects (font (size 1.27 1.27)) hide)
+    )
+    (property "Datasheet" "~" (id 3) (at 232.41 168.91 0)
+      (effects (font (size 1.27 1.27)) hide)
+    )
+    (pin "1")
+    (pin "2")
   )
   (symbol (lib_id "power:+3.3V") (at 229.87 52.07 0) (mirror y) (unit 1)
@@
     (pin "2")
   )
-  (symbol (lib_id "power:GND") (at 229.87 171.45 90) (unit 1)
-    (in_bom yes) (on_board yes)
-    (property "Reference" "#PWR0162" (id 0) (at 236.22 171.45 0)
-      (effects (font (size 1.27 1.27)) hide)
-    )
-    (property "Value" "GND" (id 1) (at 234.95 171.45 90))
-    (property "Footprint" "" (id 2) (at 229.87 171.45 0)
-      (effects (font (size 1.27 1.27)) hide)
-    )
-    (property "Datasheet" "" (id 3) (at 229.87 171.45 0)
-      (effects (font (size 1.27 1.27)) hide)
-    )
+  (symbol (lib_id "power:GND") (at 229.87 166.37 90) (unit 1)
+    (in_bom yes) (on_board yes)
+    (property "Reference" "#PWR0162" (id 0) (at 236.22 166.37 0)
+      (effects (font (size 1.27 1.27)) hide)
+    )
+    (property "Value" "GND" (id 1) (at 234.95 166.37 90))
+    (property "Footprint" "" (id 2) (at 229.87 166.37 0)
+      (effects (font (size 1.27 1.27)) hide)
+    )
+    (property "Datasheet" "" (id 3) (at 229.87 166.37 0)
+      (effects (font (size 1.27 1.27)) hide)
+    )

Commit message: Create Audio CODEC schematic block and layout.
Connections:
- net LCD_BACKGROUND_LED: now also U1.164 (PB6); no longer U1.138 (PA15)
- net RMII_TXD0: now also U1.156 (PG13); no longer U1.92 (PB12)
- net RMII_TXD1: now also U1.157 (PG14); no longer U1.93 (PB13)
- net RS485_TE: now also U1.56 (PB0); no longer U1.151 (PD7)
- net TOUCH_INT: now also U1.107 (PG3); no longer U1.134 (PI3)
Changed lines of the file:
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@@
     (effects (font (size 1.27 1.27)) (justify right))
   )
-  (hierarchical_label "LCD_BACKGROUND_LED" (shape bidirectional) (at 144.78 134.62 0)
+  (hierarchical_label "LCD_BACKGROUND_LED" (shape bidirectional) (at 144.78 154.94 0)
     (effects (font (size 1.27 1.27)) (justify left))
   )
@@
     (effects (font (size 1.27 1.27)) (justify left))
   )
-  (hierarchical_label "RS485_TE" (shape bidirectional) (at 144.78 243.84 0)
+  (hierarchical_label "RS485_TE" (shape bidirectional) (at 144.78 139.7 0)
     (effects (font (size 1.27 1.27)) (justify left))
   )
@@
     (effects (font (size 1.27 1.27)) (justify left))
   )
-  (hierarchical_label "RMII_TXD0" (shape bidirectional) (at 144.78 170.18 0)
-    (effects (font (size 1.27 1.27)) (justify left))
+  (hierarchical_label "RMII_TXD0" (shape bidirectional) (at 71.12 259.08 180)
+    (effects (font (size 1.27 1.27)) (justify right))
   )
   (hierarchical_label "LoRa_IRQ" (shape bidirectional) (at 144.78 96.52 0)
@@
     (effects (font (size 1.27 1.27)) (justify right))
   )
-  (hierarchical_label "RMII_TXD1" (shape bidirectional) (at 144.78 172.72 0)
-    (effects (font (size 1.27 1.27)) (justify left))
+  (hierarchical_label "RMII_TXD1" (shape bidirectional) (at 71.12 261.62 180)
+    (effects (font (size 1.27 1.27)) (justify right))
   )
   (hierarchical_label "I2C1_SDA" (shape bidirectional) (at 139.7 74.93 270)
@@
     (effects (font (size 1.27 1.27)) (justify left))
   )
-  (hierarchical_label "TOUCH_INT" (shape bidirectional) (at 71.12 157.48 180)
+  (hierarchical_label "TOUCH_INT" (shape bidirectional) (at 71.12 233.68 180)
     (effects (font (size 1.27 1.27)) (justify right))
   )

Commit message: Only 1 wire to complete.
Connections:
- net MCO_MCLK: now reaches U1.119 (PA8)
- net I2C2_SCL: now reaches U1.45 (PH4)
- net I2C2_SDA: now reaches U1.46 (PH5)
- net I2S2_WS: now reaches U1.92 (PB12)
- net I2S2_SCK: now reaches U1.93 (PB13)
- net I2S2_DIN: now reaches U1.94 (PB14)
- net I2S2_DOUT: now reaches U1.95 (PB15)
Other:
- moved on the sheet: C10, C11, C118, C12, C13, C14, C15, C16, C17, C18, C19, C20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
