File: RF-LORA-ZIGBEE.kicad_sch (KiCad schematic)
At the start: 3 parts, among them J4 xAnt2, J9 xAnt1, U6 Ai-Thinker-Ra-02

Commit message: Finish USB, LoRa Layout
Parts:
- removed J4: xAnt2, Anh_Footprints:Connector_Coaxial_SMA, symbol Connector:Conn_Coaxial
- removed U6: Ai-Thinker-Ra-02, RF_Module:Ai-Thinker-Ra-01-LoRa, symbol RF_Module:Ai-Thinker-Ra-02
- added C100, C101, C102, C103, C104, C105, C106, C107, C108, C109, C110, C111, C112, C113, C114, C115, C116, C91, C92, C93, C94, C95, C96, C97, C98, C99: C_Small, Capacitor_SMD:C_0603_1608Metric, symbol Device:C_Small
- added L10, L11, L12, L6, L7, L8, L9: L_Small, Inductor_SMD:L_0603_1608Metric, symbol Device:L_Small
- added Q1: BC847, Package_TO_SOT_SMD:SOT-23, symbol Transistor_BJT:BC847
- added R55, R56, R57: R_Small, Resistor_SMD:R_0603_1608Metric, symbol Device:R_Small
- added U10: MASWSS0192, Package_TO_SOT_SMD:SOT-363_SC-70-6, symbol RF_Switch:MASWSS0192
- added U6: SX1278, Package_DFN_QFN:QFN-28-1EP_6x6mm_P0.65mm_EP4.8x4.8mm, symbol RF:SX1278
- added Y4: 32MHz, Crystal:Crystal_SMD_3225-4Pin_3.2x2.5mm, symbol Device:Crystal_GND24_Small
- J9: value xAnt1 -> LoRa_Anten
Connections:
- net GND: now also C100.2, C101.2, C102.2, C104.2, C106.2, C108.1, C110.1, C112.1, C113.1, C114.1, C115.1, C116.1, C91.2, C92.1, C93.1, C94.2, C95.2, C96.2, C97.2, C98.2, C99.2, L6.2, Q1.2 (E), U10.2 (GND), U6.15 (GND), U6.21 (GND), U6.22 (GND), U6.23 (GND), U6.26 (GND), U6.29 (GND), Y4.2, Y4.4
- net at J9.1 (In): now also C116.2, L12.2
- new net: Q1.1 (B), R56.2
- new net: C113.2, Q1.3 (C), R57.1, U10.4 (V2)
- new net: C101.1, C102.1, C104.1, L9.2, U6.25 (VR_PA)
- new net: C115.2, L12.1, U10.5 (RFC)
- new net: C111.2, C112.2, L11.2, U10.3 (RF2)
- new net: C114.2, R55.2, U10.6 (V1)
- new net: C92.2, U6.5 (XTA), Y4.3
- new net: L6.1, L7.1, U6.1 (RFI_LF)
- new net: C100.1, U6.2 (VR_ANA)
- new net: R55.1, R56.1, U6.20 (RXTX/RF_MOD)
- new net: L8.1, U6.27 (PA_BOOST)
- new net: C99.1, U6.4 (VR_DIG)
- new net: C93.2, U6.6 (XTB), Y4.1
- new net: C103.1, L7.2
- new net: C105.2, U10.1 (RF1)
- new net: C107.2, C108.2, C109.1, L10.1
- new net: C109.2, C110.2, C111.1, L10.2, L11.1
- new net: C106.1, C107.1, L8.2, L9.1
- new net: C103.2, C105.1
- new net +3.3V: C91.1, C94.1, C95.1, C96.1, C97.1, C98.1, R57.2, U6.14 (VBAT_DIG), U6.24 (VBAT_RF), U6.3 (VBAT_ANA)
- new net LoRa_IRQ: U6.8 (DIO0)
- new net LoRa_MISO: U6.17 (MISO)
- new net LoRa_MOSI: U6.18 (MOSI)
- new net LoRa_NSS: U6.19 (NSS)
- new net LoRa_RST: U6.7 (~{RESET})
- new net LoRa_SCK: U6.16 (SCK)
- no-connect marks 0 -> 6
Other:
- moved on the sheet: J9
