File: RS485.kicad_sch (KiCad schematic)
At the start: 21 parts, among them J6 RS485, U8 MAX485E

Commit message: Finish SDRAM, LCD, Power block.
Connections:
- net GND: now also D7.2 (A2); no longer D7.1 (A1)
- net at D6.1 (A1), F2.1, R41.2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: now also D7.1 (A1); no longer D7.2 (A2)
Changed lines of the file:
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@@
     (pin "2")
   )
-  (symbol (lib_id "Device:D_TVS") (at 111.76 72.39 90) (unit 1)
+  (symbol (lib_id "Device:D_TVS") (at 111.76 72.39 90) (mirror x) (unit 1)
     (in_bom yes) (on_board yes) (fields_autoplaced)
     (property "Reference" "D7" (id 0) (at 114.3 71.1199 90)
