File: SDRAM.kicad_sch (KiCad schematic)
At the start: 7 parts, among them U2 IS42S16400J - HY57V641620E

Commit message: New SDRAM layout.
Parts:
- added C90: 100nF, Capacitor_SMD:C_0603_1608Metric, symbol Device:C_Small
Connections:
- net +3.3V: now also C90.2
- net GND: now also C90.1
Other:
- moved on the sheet: C44, C45, C46
