File: USB.kicad_sch (KiCad schematic)
At the start: 2 parts, among them J10 USB_OTG, J11 USB_WIFI_FLASH

Commit message: Finish SDRAM, LCD, Power block.
Parts:
- added U9: CP2102N-Axx-xQFN28, Package_DFN_QFN:QFN-28-1EP_5x5mm_P0.5mm_EP3.35x3.35mm, symbol Interface_USB:CP2102N-Axx-xQFN28
Connections:
- new net: U9.29 (GND), U9.3 (GND)
Changed lines of the file:
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@@
     (pin "S1")
+  )
+  (symbol (lib_id "Interface_USB:CP2102N-Axx-xQFN28") (at 170.18 107.95 0) (unit 1)
+    (in_bom yes) (on_board yes) (fields_autoplaced)
+    (property "Reference" "U9" (id 0) (at 172.1994 140.97 0)
+      (effects (font (size 1.27 1.27)) (justify left))
+    )
+    (property "Value" "CP2102N-Axx-xQFN28" (id 1) (at 172.1994 143.51 0)
+      (effects (font (size 1.27 1.27)) (justify left))
+    )
+    (property "Footprint" "Package_DFN_QFN:QFN-28-1EP_5x5mm_P0.5mm_EP3.35x3.35mm" (id 2) (at 203.2 139.7 0)
+      (effects (font (size 1.27 1.27)) hide)
+    )
+    (property "Datasheet" "https://www.silabs.com/documents/public/data-sheets/cp2102n-datasheet.pdf" (id 3) (at 171.45 127 0)
+      (effects (font (size 1.27 1.27)) hide)
+    )
+    (pin "1")
+    (pin "10")
+    (pin "11")
+    (pin "12")
+    (pin "13")
+    (pin "14")
+    (pin "15")
+    (pin "16")
+    (pin "17")
+    (pin "18")
+    (pin "19")
+    (pin "2")
+    (pin "20")
+    (pin "21")
+    (pin "22")
+    (pin "23")
+    (pin "24")
+    (pin "25")
+    (pin "26")
+    (pin "27")
+    (pin "28")
+    (pin "29")
+    (pin "3")
+    (pin "4")
+    (pin "5")
+    (pin "6")
+    (pin "7")
+    (pin "8")
+    (pin "9")
   )
   (symbol (lib_id "Connector:USB_C_Receptacle_USB2.0") (at 67.31 68.58 0) (unit 1)

Commit message: Finish USB, LoRa Layout
Parts:
- added C117: C_Small, Capacitor_SMD:C_0603_1608Metric, symbol Device:C_Small
- added D11, D12: SS34, Diode_SMD:D_SMA, symbol Diode:CDBA340-HF
- added Q2, Q3: BC847, Package_TO_SOT_SMD:SOT-23, symbol Transistor_BJT:BC847
- added R58, R59, R60, R61, R62, R63, R64, R65, R66, R67, R68: R_Small, Resistor_SMD:R_0603_1608Metric, symbol Device:R_Small
- added U11, U12: USBLC6-2SC6, Package_TO_SOT_SMD:SOT-23-6, symbol Power_Protection:USBLC6-2SC6
- U9: value CP2102N-Axx-xQFN28 -> CP2102N
Connections:
- net GND: now reaches J11.A1 (GND), J11.A12 (GND), J11.B1 (GND), J11.B12 (GND)
- net GND: now also J10.A1 (GND), J10.A12 (GND), J10.B1 (GND), J10.B12 (GND), J10.S1 (SHIELD), J11.S1 (SHIELD), U9.29 (GND), U9.3 (GND), C117.2, R58.2, R59.2, R63.2, R64.2, U11.2 (GND), U12.2 (GND)
- net at J11.A4 (VBUS), J11.A9 (VBUS), J11.B4 (VBUS)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: now also D12.2 (A)
- net at J11.A5 (CC1): now also R63.1
- net at J11.A6 (D+): now also J11.B6 (D+), U9.4 (D+), U12.1 (I/O1), U12.6 (I/O1)
- net at J11.A7 (D-): now also J11.B7 (D-), U9.5 (D-), U12.3 (I/O2), U12.4 (I/O2)
- net at J11.B5 (CC2): now also R64.1
- net at U9.24 (~{RTS}): now also Q3.2 (E), R67.2
- net RXD: now reaches U9.25 (RXD)
- net at U9.26 (TXD): now also R66.2
- net at U9.28 (~{DTR}): now also Q2.2 (E), R68.2
- net at U9.6 (VDD): now also C117.1
- net +5V: now reaches U9.7 (VREGIN)
- net +5V: now also U9.8 (VBUS), D11.1 (K), D12.1 (K), R65.2, U11.5 (VBUS), U12.5 (VBUS)
- net at U9.9 (~{RST}): now also R65.1
- net at J10.A4 (VBUS), J10.A9 (VBUS), J10.B4 (VBUS)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: now also D11.2 (A)
- net at J10.A5 (CC1): now also R58.1
- net at J10.A6 (D+): now also J10.B6 (D+), R60.1, R62.1, U11.3 (I/O2), U11.4 (I/O2)
- net at J10.A7 (D-): now also J10.B7 (D-), R61.1, U11.1 (I/O1), U11.6 (I/O1)
- net at J10.B5 (CC2): now also R59.1
- new net: Q2.1 (B), R67.1
- new net: Q3.1 (B), R68.1
- new net +3.3V: R60.2
- new net OTG_DM: R61.2
- new net OTG_DP: R62.2
- new net TXD: R66.1
- new net WiFi_BOOT: Q3.3 (C)
- new net WiFi_RST: Q2.3 (C)
- no-connect marks 0 -> 20
Other:
- moved on the sheet: J10, J11, U9
