File: WIFI.kicad_sch (KiCad schematic)
At the start: 33 parts, among them J3 ESP Anten, SW2 ESP_RESET, SW3 ESP_BOOT, U4 ESP32-D0WD-V3, U5 W25Q32JVSS, Y3 40MHz

Commit message: Finish SDRAM, LCD, Power block.
Parts:
- added C89: 10uF, Capacitor_SMD:C_1206_3216Metric, symbol Device:C_Small
Connections:
- net +3.3V: now also C89.2
- net GND: now also C89.1
Changed lines of the file:
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@@
   (junction (at 154.94 152.4) (diameter 0) (color 0 0 0 0)
   )
+  (junction (at 49.53 46.99) (diameter 0) (color 0 0 0 0)
+  )
   (junction (at 73.66 68.58) (diameter 0) (color 0 0 0 0)
   )
   (junction (at 111.76 58.42) (diameter 0) (color 0 0 0 0)
+  )
+  (junction (at 49.53 54.61) (diameter 0) (color 0 0 0 0)
   )
   (junction (at 129.54 139.7) (diameter 0) (color 0 0 0 0)
@@
     (stroke (width 0) (type default) (color 0 0 0 0))
   )
+  (wire (pts (xy 53.34 48.26) (xy 53.34 46.99))
+    (stroke (width 0) (type default) (color 0 0 0 0))
+  )
   (wire (pts (xy 161.29 111.76) (xy 153.67 111.76))
     (stroke (width 0) (type default) (color 0 0 0 0))
@@
     (stroke (width 0) (type default) (color 0 0 0 0))
   )
+  (wire (pts (xy 49.53 54.61) (xy 53.34 54.61))
+    (stroke (width 0) (type default) (color 0 0 0 0))
+  )
   (wire (pts (xy 59.69 121.92) (xy 55.88 121.92))
     (stroke (width 0) (type default) (color 0 0 0 0))
@@
     (stroke (width 0) (type default) (color 0 0 0 0))
   )
+  (wire (pts (xy 53.34 46.99) (xy 49.53 46.99))
+    (stroke (width 0) (type default) (color 0 0 0 0))
+  )
   (wire (pts (xy 104.14 58.42) (xy 105.41 58.42))
     (stroke (width 0) (type default) (color 0 0 0 0))
@@
   )
   (wire (pts (xy 123.19 52.07) (xy 123.19 44.45))
+    (stroke (width 0) (type default) (color 0 0 0 0))
+  )
+  (wire (pts (xy 53.34 54.61) (xy 53.34 53.34))
     (stroke (width 0) (type default) (color 0 0 0 0))
   )
@@
     (pin "1")
   )
+  (symbol (lib_id "Device:C_Small") (at 53.34 50.8 180) (unit 1)
+    (in_bom yes) (on_board yes)
+    (property "Reference" "C89" (id 0) (at 52.07 53.34 90))
+    (property "Value" "10uF" (id 1) (at 52.07 45.72 90))
+    (property "Footprint" "Capacitor_SMD:C_1206_3216Metric" (id 2) (at 53.34 50.8 0)
+      (effects (font (size 1.27 1.27)) hide)
+    )
+    (property "Datasheet" "~" (id 3) (at 53.34 50.8 0)
+      (effects (font (size 1.27 1.27)) hide)
+    )
+    (pin "1")
+    (pin "2")
+  )
   (symbol (lib_id "power:GND") (at 95.25 58.42 270) (unit 1)

Commit message: Finish USB, LoRa Layout
Connections:
- net WiFi_RST: now reaches C25.2, R17.1, SW2.2, U4.9 (CHIP_PU)
Changed lines of the file:
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@@
+    (stroke (width 0) (type default) (color 0 0 0 0))
+  )
+  (wire (pts (xy 62.23 109.22) (xy 63.5 109.22))
     (stroke (width 0) (type default) (color 0 0 0 0))
   )
@@
     (effects (font (size 1.27 1.27)) (justify left))
   )
+  (hierarchical_label "WiFi_RST" (shape bidirectional) (at 63.5 109.22 0)
+    (effects (font (size 1.27 1.27)) (justify left))
+  )
