File: POWER.kicad_sch (KiCad schematic)
At the start: 39 parts, among them IC1 MP1584EN, IC2 MP1584EN, J7 Conn_Jack-DC

Commit message: Power route bug.
Parts:
- added JP15: 3V3_SW, Jumper:SolderJumper-3_P1.3mm_Open_Pad1.0x1.5mm_NumberLabels, symbol Jumper:SolderJumper_3_Open
Connections:
- net +5V: now also JP15.3 (B)
- net VCC: now also JP15.1 (A); no longer C85.2, IC1.7 (VIN), R43.1
- new net: C85.2, IC1.7 (VIN), JP15.2 (C), R43.1
Changed lines of the file:
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@@
+    )
+  )
+  (symbol (lib_id "Jumper:SolderJumper_3_Open") (at 116.84 36.83 0) (unit 1)
+    (in_bom yes) (on_board yes) (dnp no)
+    (property "Reference" "JP15" (at 116.84 31.75 0)
+      (effects (font (size 1.27 1.27)))
+    )
+    (property "Value" "3V3_SW" (at 116.84 34.29 0)
+      (effects (font (size 1.27 1.27)))
+    )
+    (property "Footprint" "Jumper:SolderJumper-3_P1.3mm_Open_Pad1.0x1.5mm_NumberLabels" (at 116.84 36.83 0)
+      (effects (font (size 1.27 1.27)) hide)
+    )
+    (property "Datasheet" "~" (at 116.84 36.83 0)
+      (effects (font (size 1.27 1.27)) hide)
+    )
+    (pin "1")
+    (pin "2")
+    (pin "3")
+    (instances
+      (project "GatewayPlus_V1.1"
+        (path "/6b25bb2e-e3f8-49e6-940a-fa3f985570a5/4931c4f2-ec98-49ed-98f1-a79587b46d92"
+          (reference "JP15") (unit 1)
+        )
+      )
     )
   )
@@
         (path "/6b25bb2e-e3f8-49e6-940a-fa3f985570a5/4931c4f2-ec98-49ed-98f1-a79587b46d92"
           (reference "JP13") (unit 1)
+        )
+      )
+    )
+  )
+  (symbol (lib_id "power:+5V") (at 121.92 36.83 0) (unit 1)
+    (in_bom yes) (on_board yes) (dnp no)
+    (property "Reference" "#PWR030" (at 121.92 40.64 0)
+      (effects (font (size 1.27 1.27)) hide)
+    )
+    (property "Value" "+5V" (at 119.38 33.02 0)
+      (effects (font (size 1.27 1.27)) (justify left))
+    )
+    (property "Footprint" "" (at 121.92 36.83 0)
+      (effects (font (size 1.27 1.27)) hide)
+    )
+    (property "Datasheet" "" (at 121.92 36.83 0)
+      (effects (font (size 1.27 1.27)) hide)
+    )
+    (pin "1")
+    (instances
+      (project "GatewayPlus_V1.1"
+        (path "/6b25bb2e-e3f8-49e6-940a-fa3f985570a5/4931c4f2-ec98-49ed-98f1-a79587b46d92"
+          (reference "#PWR030") (unit 1)
         )
       )
@@
     )
   )
-  (symbol (lib_id "power:VCC") (at 116.84 40.64 0) (unit 1)
-    (in_bom yes) (on_board yes) (dnp no) (fields_autoplaced)
-    (property "Reference" "#PWR0202" (at 116.84 44.45 0)
-      (effects (font (size 1.27 1.27)) hide)
-    )
-    (property "Value" "VCC" (at 116.84 35.56 0)
-      (effects (font (size 1.27 1.27)))
-    )
-    (property "Footprint" "" (at 116.84 40.64 0)
-      (effects (font (size 1.27 1.27)) hide)
-    )
-    (property "Datasheet" "" (at 116.84 40.64 0)
-      (effects (font (size 1.27 1.27)) hide)
-    )
+  (symbol (lib_id "power:VCC") (at 111.76 36.83 0) (unit 1)
+    (in_bom yes) (on_board yes) (dnp no) (fields_autoplaced)
+    (property "Reference" "#PWR0202" (at 111.76 40.64 0)
+      (effects (font (size 1.27 1.27)) hide)
+    )
+    (property "Value" "VCC" (at 111.76 31.75 0)
+      (effects (font (size 1.27 1.27)))
+    )
+    (property "Footprint" "" (at 111.76 36.83 0)
+      (effects (font (size 1.27 1.27)) hide)
+    )
+    (property "Datasheet" "" (at 111.76 36.83 0)
+      (effects (font (size 1.27 1.27)) hide)
+    )
